File: hardware/kicad/usb_lan.kicad_sch (KiCad schematic)
At the start: 24 parts, among them J1 USB-C (USB2.0), SW1 RESET, SW2 BOOT, U1 ESP32-S3-WROOM-1U-N8R2, U2 USBLC6-2SC6, U3 AP2112K-3.3

Commit message: Add FM transmitter I/F header (FPGA/ADF4002), status LED; rev 0.2
- J2 2x8 header: FPGA UART1 (GPIO17/18) + RST (GPIO4), ADF4002 3-wire
  CLK/DATA/LE (GPIO10/11/12) + MUXOUT lock detect (GPIO6), TX_EN (GPIO5),
  ADC (GPIO1), spare I2C (GPIO8/9, 4.7k pull-ups), +3V3/+5V/GND
- Status LED on GPIO21 (lit while Wi-Fi link is up)
- firmware/main/board_pins.h mirrors the schematic pin assignment
- Netlist verified with kicad-cli; NCM build passes

Co-Authored-By: Claude Opus 5.5 <noreply@anthropic.com>
Claude-Session: https://claude.ai/code/session_01Ls5zZCBa6fHzoAG8K7unes
Parts:
- added D1: LED 緑, LED_SMD:LED_0603_1608Metric, symbol usb_lan:LED
- added J2: FM I/F, Connector_PinHeader_2.54mm:PinHeader_2x08_P2.54mm_Vertical, symbol usb_lan:Conn_02x08
- added R7, R8: 4.7k, Resistor_SMD:R_0603_1608Metric, symbol usb_lan:R
- added R9: 1k, Resistor_SMD:R_0603_1608Metric, symbol usb_lan:R
Connections:
- net +3V3: now also J2.1 (+3V3), R7.1, R8.1
- net +5V: now also J2.2 (+5V)
- net GND: now also D1.1, J2.16 (GND), J2.3 (GND), J2.4 (GND)
- net FPGA_TXD: now reaches U1.10 (IO17)
- net FPGA_TXD: now also J2.7 (TXD)
- net FPGA_RXD: now reaches U1.11 (IO18)
- net FPGA_RXD: now also J2.8 (RXD)
- net I2C_SDA: now reaches U1.12 (IO8)
- net I2C_SDA: now also J2.5 (SDA), R7.2
- net I2C_SCL: now reaches U1.17 (IO9)
- net I2C_SCL: now also J2.6 (SCL), R8.2
- net ADF_CLK: now reaches U1.18 (IO10)
- net ADF_CLK: now also J2.13 (CLK)
- net ADF_DATA: now reaches U1.19 (IO11)
- net ADF_DATA: now also J2.14 (DATA)
- net ADF_LE: now reaches U1.20 (IO12)
- net ADF_LE: now also J2.15 (LE)
- net LED_DRV: now reaches U1.23 (IO21)
- net LED_DRV: now also R9.1
- net FM_ADC: now reaches U1.39 (IO1)
- net FM_ADC: now also J2.12 (ADC)
- net FPGA_RST: now reaches U1.4 (IO4)
- net FPGA_RST: now also J2.9 (RST)
- net FM_TX_EN: now reaches U1.5 (IO5)
- net FM_TX_EN: now also J2.10 (EN)
- net ADF_MUXOUT: now reaches U1.6 (IO6)
- net ADF_MUXOUT: now also J2.11 (MUX)
- new net LED_A: D1.2, R9.2
- no-connect marks 34 -> 22
Other:
- note added: "J2: 送信機 (FM) 接続用 拡張ヘッダ (3.3V ロジック) ・I2C: SDA=GPIO8 / SCL=GPIO9 (4.7k プルアップ) ・FPGA: UART1 TXD=GPIO17 / RXD=GPIO18, RST=GPIO4 ・ADF4002: CLK=GPIO10 / DATA=GPIO11 / LE=GPIO12, MUXOUT=GPIO6 ・TX_EN=GPIO5 (RF 出力 ON/OFF), ADC=GPIO1 (RF レベル) ・+5V は PTC の後 (USB 給電 0.5A を ESP32 と共用) ・5V ロジックの送信機はレベル変換が必要"
- note added: "状態 LED: GPIO21 (High で点灯)"

Commit message: Switch FPGA link to 4-wire SPI (Rev.B2) on SPI2 IO_MUX pins; rev 0.3
- J2: MISO=GPIO13 (pin 7), FPGA_CS=GPIO10 (pin 8), SCK=GPIO12 (pin 13),
  MOSI=GPIO11 (pin 14); ADF4002 shares SCK/MOSI with its own LE=GPIO14
  (pin 15); UART1 on GPIO17/18 removed from the header
- board_pins.h updated (BOARD_SPI_*, BOARD_FPGA_CS, BOARD_ADF_LE)
- Netlist verified with kicad-cli; NCM build passes

Co-Authored-By: Claude Opus 5.5 <noreply@anthropic.com>
Claude-Session: https://claude.ai/code/session_01Ls5zZCBa6fHzoAG8K7unes
Connections:
- net ADF_LE: now also U1.22 (IO14); no longer U1.20 (IO12)
- net SPI_MISO: now reaches U1.21 (IO13)
- net SPI_MISO: now also J2.7 (MISO)
- net ADF_CLK renamed FPGA_CS
- net FPGA_CS: now also J2.8 (CS); no longer J2.13 (CLK)
- net ADF_DATA renamed SPI_MOSI
- net FPGA_RXD: no longer names the net of U1.11 (IO18)
- net FPGA_RXD: no longer J2.8 (RXD)
- net FPGA_TXD: no longer names the net of U1.10 (IO17)
- net FPGA_TXD: no longer J2.7 (TXD)
- new net SPI_SCK: J2.13 (SCK), U1.20 (IO12)
Other:
- note added: "J2: 送信機 (FM) 接続用 拡張ヘッダ (3.3V ロジック) ・I2C: SDA=GPIO8 / SCL=GPIO9 (4.7k プルアップ) ・SPI2 (IO_MUX): SCK=GPIO12 / MOSI=GPIO11 / MISO=GPIO13 ・FPGA: CS=GPIO10, RST=GPIO4 / ADF4002: SCK・MOSI 共用, LE=GPIO14, MUXOUT=GPIO6 ・TX_EN=GPIO5 (RF 出力 ON/OFF), ADC=GPIO1 (RF レベル) ・+5V は PTC の後 (USB 給電 0.5A を ESP32 と共用) ・5V ロジックの送信機はレベル変換が必要"
- note removed: "J2: 送信機 (FM) 接続用 拡張ヘッダ (3.3V ロジック) ・I2C: SDA=GPIO8 / SCL=GPIO9 (4.7k プルアップ) ・FPGA: UART1 TXD=GPIO17 / RXD=GPIO18, RST=GPIO4 ・ADF4002: CLK=GPIO10 / DATA=GPIO11 / LE=GPIO12, MUXOUT=GPIO6 ・TX_EN=GPIO5 (RF 出力 ON/OFF), ADC=GPIO1 (RF レベル) ・+5V は PTC の後 (USB 給電 0.5A を ESP32 と共用) ・5V ロジックの送信機はレベル変換が必要"
Changed lines of the file:
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@@
 (kicad_sch (version 20230121) (generator eeschema)
   (paper "A3")
-  (title_block (title "USB-LAN adapter (ESP32-S3-WROOM-1U / USB CDC-NCM)") (date "2026-10-01") (rev "0.2") (comment 1 "Initial draft - generated by hardware/tools/gen_schematic.py"))
+  (title_block (title "USB-LAN adapter (ESP32-S3-WROOM-1U / USB CDC-NCM)") (date "2026-10-01") (rev "0.3") (comment 1 "Initial draft - generated by hardware/tools/gen_schematic.py"))
   (symbol (lib_id "usb_lan:USB_C_USB2.0_16P") (at 40.64 71.12 0) (unit 1)
     (in_bom yes) (on_board yes) (dnp no)
@@
   (label "I2C_SCL" (at 322.58 100.33 270) (fields_autoplaced) (effects (font (size 1.27 1.27)) (justify left bottom)))
   (label "I2C_SCL" (at 354.33 114.3 0) (fields_autoplaced) (effects (font (size 1.27 1.27)) (justify left bottom)))
-  (label "FPGA_TXD" (at 266.7 101.6 0) (fields_autoplaced) (effects (font (size 1.27 1.27)) (justify left bottom)))
-  (label "FPGA_TXD" (at 336.55 116.84 180) (fields_autoplaced) (effects (font (size 1.27 1.27)) (justify right bottom)))
-  (label "FPGA_RXD" (at 266.7 104.14 0) (fields_autoplaced) (effects (font (size 1.27 1.27)) (justify left bottom)))
-  (label "FPGA_RXD" (at 354.33 116.84 0) (fields_autoplaced) (effects (font (size 1.27 1.27)) (justify left bottom)))
+  (label "SPI_MISO" (at 266.7 91.44 0) (fields_autoplaced) (effects (font (size 1.27 1.27)) (justify left bottom)))
+  (label "SPI_MISO" (at 336.55 116.84 180) (fields_autoplaced) (effects (font (size 1.27 1.27)) (justify right bottom)))
+  (label "FPGA_CS" (at 266.7 83.82 0) (fields_autoplaced) (effects (font (size 1.27 1.27)) (justify left bottom)))
+  (label "FPGA_CS" (at 354.33 116.84 0) (fields_autoplaced) (effects (font (size 1.27 1.27)) (justify left bottom)))
   (label "FPGA_RST" (at 241.3 121.92 180) (fields_autoplaced) (effects (font (size 1.27 1.27)) (justify right bottom)))
   (label "FPGA_RST" (at 336.55 119.38 180) (fields_autoplaced) (effects (font (size 1.27 1.27)) (justify right bottom)))
@@
   (label "FM_ADC" (at 241.3 116.84 180) (fields_autoplaced) (effects (font (size 1.27 1.27)) (justify right bottom)))
   (label "FM_ADC" (at 354.33 121.92 0) (fields_autoplaced) (effects (font (size 1.27 1.27)) (justify left bottom)))
-  (label "ADF_CLK" (at 266.7 83.82 0) (fields_autoplaced) (effects (font (size 1.27 1.27)) (justify left bottom)))
-  (label "ADF_CLK" (at 336.55 124.46 180) (fields_autoplaced) (effects (font (size 1.27 1.27)) (justify right bottom)))
-  (label "ADF_DATA" (at 266.7 86.36 0) (fields_autoplaced) (effects (font (size 1.27 1.27)) (justify left bottom)))
-  (label "ADF_DATA" (at 354.33 124.46 0) (fields_autoplaced) (effects (font (size 1.27 1.27)) (justify left bottom)))
-  (label "ADF_LE" (at 266.7 88.9 0) (fields_autoplaced) (effects (font (size 1.27 1.27)) (justify left bottom)))
+  (label "SPI_SCK" (at 266.7 88.9 0) (fields_autoplaced) (effects (font (size 1.27 1.27)) (justify left bottom)))
+  (label "SPI_SCK" (at 336.55 124.46 180) (fields_autoplaced) (effects (font (size 1.27 1.27)) (justify right bottom)))
+  (label "SPI_MOSI" (at 266.7 86.36 0) (fields_autoplaced) (effects (font (size 1.27 1.27)) (justify left bottom)))
+  (label "SPI_MOSI" (at 354.33 124.46 0) (fields_autoplaced) (effects (font (size 1.27 1.27)) (justify left bottom)))
+  (label "ADF_LE" (at 266.7 93.98 0) (fields_autoplaced) (effects (font (size 1.27 1.27)) (justify left bottom)))
   (label "ADF_LE" (at 336.55 127 180) (fields_autoplaced) (effects (font (size 1.27 1.27)) (justify right bottom)))
   (label "LED_DRV" (at 266.7 106.68 0) (fields_autoplaced) (effects (font (size 1.27 1.27)) (justify left bottom)))
@@
   (no_connect (at 241.3 119.38))
   (no_connect (at 241.3 129.54))
-  (no_connect (at 266.7 91.44))
-  (no_connect (at 266.7 93.98))
   (no_connect (at 266.7 96.52))
   (no_connect (at 266.7 99.06))
+  (no_connect (at 266.7 101.6))
+  (no_connect (at 266.7 104.14))
   (no_connect (at 266.7 109.22))
   (no_connect (at 266.7 111.76))
@@
   (text "EN: 10k/1uF の RC 遅延 + RESET スイッチ\nIO0: BOOT スイッチ (内部プルアップ)\n書込み: BOOT 押しながら RESET → ROM の USB-Serial/JTAG で idf.py flash" (at 180.34 190.5 0) (effects (font (size 1.524 1.524)) (justify left top)))
   (text "UART0 テストパッド (ログ/予備書込み)" (at 317.5 38.1 0) (effects (font (size 1.524 1.524)) (justify left top)))
-  (text "J2: 送信機 (FM) 接続用 拡張ヘッダ (3.3V ロジック)\n・I2C: SDA=GPIO8 / SCL=GPIO9 (4.7k プルアップ)\n・FPGA: UART1 TXD=GPIO17 / RXD=GPIO18, RST=GPIO4\n・ADF4002: CLK=GPIO10 / DATA=GPIO11 / LE=GPIO12, MUXOUT=GPIO6\n・TX_EN=GPIO5 (RF 出力 ON/OFF), ADC=GPIO1 (RF レベル)\n・+5V は PTC の後 (USB 給電 0.5A を ESP32 と共用)\n・5V ロジックの送信機はレベル変換が必要" (at 297.18 66.04 0) (effects (font (size 1.524 1.524)) (justify left top)))
+  (text "J2: 送信機 (FM) 接続用 拡張ヘッダ (3.3V ロジック)\n・I2C: SDA=GPIO8 / SCL=GPIO9 (4.7k プルアップ)\n・SPI2 (IO_MUX): SCK=GPIO12 / MOSI=GPIO11 / MISO=GPIO13\n・FPGA: CS=GPIO10, RST=GPIO4 / ADF4002: SCK・MOSI 共用, LE=GPIO14, MUXOUT=GPIO6\n・TX_EN=GPIO5 (RF 出力 ON/OFF), ADC=GPIO1 (RF レベル)\n・+5V は PTC の後 (USB 給電 0.5A を ESP32 と共用)\n・5V ロジックの送信機はレベル変換が必要" (at 297.18 66.04 0) (effects (font (size 1.524 1.524)) (justify left top)))
   (text "状態 LED: GPIO21 (High で点灯)" (at 297.18 152.4 0) (effects (font (size 1.524 1.524)) (justify left top)))
   (sheet_instances (path "/" (page "1")))

Commit message: Board rev 0.4: add J3 for loop-filter / MPX control and boot-time pull resistors
J3 carries LF_INPUT_SEL, LF_FB_SEL, LF_PRECHARGE, MPX_RUN, MPX_MUTE and ADF_CE
(GPIO15/16/17/18/7/2). R10-R15 hold the transmitter muted, RF off, loop in
ACQUIRE and the PLL powered down while the ESP32-S3 pins are still floating.

Co-Authored-By: Claude Opus 5.5 <noreply@anthropic.com>
Parts:
- added J3: FM LOOP, Connector_PinHeader_2.54mm:PinHeader_2x04_P2.54mm_Vertical, symbol usb_lan:Conn_02x04
- added R10, R11, R12, R13, R14, R15: 10k, Resistor_SMD:R_0603_1608Metric, symbol usb_lan:R
Connections:
- net +3V3: now also J3.7 (+3V3), R10.2, R11.2, R13.2
- net FM_TX_EN: now also R15.1
- net GND: now also J3.8 (GND), R12.2, R14.2, R15.2
- net LF_PRECHARGE: now reaches U1.10 (IO17)
- net LF_PRECHARGE: now also J3.3 (LF_PRE)
- net MPX_RUN: now reaches U1.11 (IO18)
- net MPX_RUN: now also J3.4 (MPX_RUN), R12.1
- net ADF_CE: now reaches U1.38 (IO2)
- net ADF_CE: now also J3.6 (ADF_CE), R14.1
- net MPX_MUTE: now reaches U1.7 (IO7)
- net MPX_MUTE: now also J3.5 (MPX_MUTE), R13.1
- net LF_INPUT_SEL: now reaches U1.8 (IO15)
- net LF_INPUT_SEL: now also J3.1 (LF_IN), R10.1
- net LF_FB_SEL: now reaches U1.9 (IO16)
- net LF_FB_SEL: now also J3.2 (LF_FB), R11.1
- no-connect marks 22 -> 16
Other:
- note added: "J2: 送信機 (FM) 接続用 拡張ヘッダ (3.3V ロジック) ・I2C: SDA=GPIO8 / SCL=GPIO9 (4.7k プルアップ) ・SPI2 (IO_MUX): SCK=GPIO12 / MOSI=GPIO11 / MISO=GPIO13 ・FPGA: CS=GPIO10, RST=GPIO4 (High でリセット) / ADF4002: SCK・MOSI 共用, LE=GPIO14, MUXOUT=GPIO6 ・TX_EN=GPIO5 (RF 出力 ON/OFF), ADC=GPIO1 (RF レベル) ・+5V は PTC の後 (USB 給電 0.5A を ESP32 と共用) ・5V ロジックの送信機はレベル変換が必要"
- note added: "J3 (rev 0.4): 切替式ループフィルタ / MPX 制御 (3.3V ロジック, TMUX1136 の SEL へ) ・LF_INPUT_SEL=GPIO15 / LF_FB_SEL=GPIO16 (1 = ACQUIRE), LF_PRECHARGE=GPIO17 ・MPX_RUN=GPIO18, MPX_MUTE=GPIO7 (FPGA へ), ADF_CE=GPIO2 ・R10-R15: 起動中 (ピンがハイインピーダンスの間) は ミュート・RF OFF・ACQUIRE・PLL 停止"
- note removed: "J2: 送信機 (FM) 接続用 拡張ヘッダ (3.3V ロジック) ・I2C: SDA=GPIO8 / SCL=GPIO9 (4.7k プルアップ) ・SPI2 (IO_MUX): SCK=GPIO12 / MOSI=GPIO11 / MISO=GPIO13 ・FPGA: CS=GPIO10, RST=GPIO4 / ADF4002: SCK・MOSI 共用, LE=GPIO14, MUXOUT=GPIO6 ・TX_EN=GPIO5 (RF 出力 ON/OFF), ADC=GPIO1 (RF レベル) ・+5V は PTC の後 (USB 給電 0.5A を ESP32 と共用) ・5V ロジックの送信機はレベル変換が必要"
